File: hand_pnp.kicad_pcb (KiCad board)
At the start: 2 copper layers, 46 x 41 mm, 16 parts, among them J1 Solenoid, J2 Motor, J3 12v in, J4 AudioJack3_Ground, Q1 FDN339AN, Q2 FDN339AN, SW1 power sw

Commit message: Added renders, readme and gerbers
Parts:
- added G***: LOGO, graphics:kiwi12.5mm, B.Cu at (148.0, 49.0)
Routing:
- net +12V: track 59.2 -> 61.9 mm
- net GND: track 71.5 -> 69.2 mm
- net /motor_E: track 22.3 -> 21.2 mm
Other:
- board text added: "(3,3) (0,0)"
- board text added: "(43,3) (40,0)"
- board text added: "(43,38) ( 0,35)"
- board text added: "(43,38) (40,35)"
- board text added: "Mounting hole position is given in two ways (0,0) = top left board edge (0,0) = top left hole (seen from the top)"
